Commit message: fixed urdf, CAN hw_info and ros2 control

File: src/grr_description/urdf/parts/chassis.xacro (robot description, xacro)
@@ -1,16 +1,15 @@
 <?xml version="1.0" ?>
 <robot xmlns:xacro="http://www.ros.org/wiki/xacro">
-  <xacro:macro name="chassis" params="length width height mass">
-    <link name="base_link"></link>
+  <xacro:macro name="chassis" params="parent *origin length width height mass">
     <link name="chassis_link">
-      <xacro:inertial_box mass="${chassis_weight}" x="${length}" y="${width}" z="${height}">
-        <origin xyz="0 0 -${height / 2}" rpy="0 0 0"/>
+      <xacro:inertial_box mass="${mass}" x="${length}" y="${width}" z="${height}">
+        <origin xyz="0 0 0" rpy="0 0 0"/>
       </xacro:inertial_box>
       <visual>
-        <origin xyz="0 0 0" rpy="0 0 0"/>
+        <origin xyz="0 0 0" rpy="0 0 ${M_PI}"/>
         <geometry>
-          <mesh filename="package://grr_description/meshes/slim_drivebase.stl" scale="0.001 0.001 0.001"/>
+          <mesh filename="package://grr_description/meshes/drivebase.stl" scale="1 1 1"/>
         </geometry>
-        <material name="blue"/>
+        <!-- <material name="blue"/> -->
       </visual>
       <collision>
@@ -21,11 +20,8 @@
       </collision>
     </link>
-    <gazebo reference="chassis">
-      <material>Gazebo/Blue</material>
-    </gazebo>
     <joint name="chassis_joint" type="fixed">
       <parent link="base_link"/>
       <child link="chassis_link"/>
-      <origin xyz="0 0 0"/>
+      <xacro:insert_block name="origin" />
     </joint>
   </xacro:macro>

File: src/grr_description/urdf/parts/mecanum_roller.xacro (robot description, xacro)
@@ -3,15 +3,15 @@
   <xacro:macro name="roller" params="name number">
     <!-- Type Offset: When type 1 output 1. When type 2 output -1 -->
-    <xacro:property name="type_offset" value="${(type * 2 - 3) * -1}" />
+    <xacro:property name="type_offset" value="${(type * 2 - 3) }" />
     <!-- Compute incremental radians to place the roller around the hub -->
     <xacro:property name="roller_radians" value="${(2 * pi / roller_total * number)}" />
     <!-- Figure out the x and y position of the roller from radian value -->
     <xacro:property name="roller_x_pos" value="${sin(roller_radians) * wheel_radius}" />
-    <xacro:property name="roller_y_pos" value="${cos(roller_radians) * wheel_radius}" />
+    <xacro:property name="roller_z_pos" value="${cos(roller_radians) * wheel_radius}" />
     <!-- Figure out how much to rotate a roller. It should be angled 45 degrees -->
     <xacro:property name="roller_x_rot" value="${sin(roller_radians) * (pi/4) * type_offset}" />
     <xacro:property name="roller_y_rot" value="${cos(roller_radians) * (pi/4) * type_offset}" />
     <xacro:property name="roller_z_rot" value="0"/>
-    <xacro:if value="${number==1}">
+    <!-- <xacro:if value="${number==1}">
     </xacro:if>
     <xacro:if value="${number==3}">
@@ -23,8 +23,8 @@
       <xacro:property name="roller_y_rot" value="${(cos(roller_radians) * (pi/4) * type_offset)+(3.095*pi/180)}" />
       <xacro:property name="roller_z_rot" value="${(5.395*pi/180)}"/>
-    </xacro:if>
+    </xacro:if> -->
     <link name="${name}_roller_${number}">
       <visual>
-        <origin xyz="0 0 0" rpy="0 0 0"/>
+        <origin xyz="0 0 0" rpy="0 0 -${M_PI/2} "/>
         <geometry>
           <mesh filename="package://grr_description/meshes/mecanum_roller.stl" scale="0.001 0.001 0.001"/>
@@ -32,34 +32,4 @@
         <material name="grey"/>
       </visual>
-      <!-- <collision>
-        <origin xyz="0 0 0" rpy="0 0 0"/>
-        <geometry>
-          <sphere radius="${roller_middle_radius}"/>
-        </geometry>
-      </collision>
-      <collision>
-        <origin xyz="0 0 ${roller_length/5}" rpy="0 0 0"/>
-        <geometry>
-          <sphere radius="${roller_second_radius}"/>
-        </geometry>
-      </collision>
-      <collision>
-        <origin xyz="0 0 -${roller_length/5}" rpy="0 0 0"/>
-        <geometry>
-          <sphere radius="${roller_second_radius}"/>
-        </geometry>
-      </collision>
-      <collision>
-        <origin xyz="0 0 ${2 * roller_length/5}" rpy="0 0 0"/>
-        <geometry>
-          <sphere radius="${roller_third_radius}"/>
-        </geometry>
-      </collision>
-      <collision>
-        <origin xyz="0 0 -${2 * roller_length/5}" rpy="0 0 0"/>
-        <geometry>
-          <sphere radius="${roller_third_radius}"/>
-        </geometry>
-      </collision> -->
       <collision>
         <origin xyz="0 0 0" rpy="0 0 0"/>
@@ -73,5 +43,5 @@
     </link>
     <joint name="${name}_roller_${number}_joint" type="continuous">
-      <origin xyz="${roller_x_pos} ${roller_y_pos} 0" rpy="${roller_x_rot} ${roller_y_rot} ${roller_z_rot}"/>
+      <origin xyz="${roller_x_pos} 0 ${roller_z_pos}" rpy="${roller_x_rot} ${roller_z_rot} ${roller_y_rot}"/>
       <parent link="${name}_mecanum_link"/>
       <child link="${name}_roller_${number}"/>

File: src/grr_description/urdf/parts/mecanum_wheel.xacro (robot description, xacro)
@@ -24,5 +24,5 @@
       <parent link="chassis_link"/>
       <child link="${name}_mecanum_link"/>
-      <axis xyz="0.0 0.0 ${copysign(1, (flip * -1))}"/>
+      <axis xyz="0.0 ${copysign(1, (flip * -1))} 0.0 "/>
     </joint>
     <!-- There will be 8 rollers for each wheel -->

File: src/grr_description/urdf/parts/zed_cam.xacro (robot description, xacro)
@@ -51,5 +51,5 @@
     </joint>
     <!-- Right Camera -->
-    <link name="zed_right_camera_frame" />
+    <link name="zed_right_camera_frame" />      //call assign id function
     <joint name="zed_right_camera_joint" type="fixed">
       <parent link="zed_camera_center"/>

File: src/grr_description/urdf/util/materials.xacro (robot description, xacro)
@@ -1,37 +1,66 @@
 <?xml version="1.0"?>
-<!--
-Copied from ROS1 example:
-https://github.com/ros-simulation/gazebo_ros_demos/blob/kinetic-devel/rrbot_description/urdf/materials.xacro
--->
 <robot>
   <material name="black">
-    <color rgba="0.0 0.0 0.0 1.0"/>
+    <color rgba="0.0 0.0 0.0 1.0" />
   </material>
   <material name="blue">
-    <color rgba="${35/255} ${110/255} ${150/255} 1.0"/>
+    <color rgba="${35/255} ${110/255} ${150/255} 1.0" />
   </material>
   <material name="green">
-    <color rgba="0.0 0.8 0.0 1.0"/>
+    <color rgba="0.0 0.8 0.0 1.0" />
   </material>
   <material name="grey">
-    <color rgba="0.2 0.2 0.2 1.0"/>
+    <color rgba="0.2 0.2 0.2 1.0" />
   </material>
   <material name="yellow">
-    <color rgba="${255/255} ${215/255} ${0/255} 1"/>
+    <color rgba="${255/255} ${215/255} ${0/255} 1" />
   </material>
   <material name="orange">
-    <color rgba="${243/255} ${135/255} ${47/255} 1"/>
+    <color rgba="${243/255} ${135/255} ${47/255} 1" />
   </material>
   <material name="brown">
-    <color rgba="${222/255} ${207/255} ${195/255} 1.0"/>
+    <color rgba="${222/255} ${207/255} ${195/255} 1.0" />
   </material>
   <material name="red">
-    <color rgba="0.8 0.0 0.0 1.0"/>
+    <color rgba="0.8 0.0 0.0 1.0" />
   </material>
   <material name="white">
-    <color rgba="1.0 1.0 1.0 1.0"/>
+    <color rgba="1.0 1.0 1.0 1.0" />
   </material>
   <material name="silver">
-    <color rgba="0.700 0.700 0.700 1.000"/>
+    <color rgba="0.700 0.700 0.700 1.000" />
+  </material>
+  <material name="aluminum">
+    <color rgba="0.5 0.5 0.5 1" />
+  </material>
+  <material name="plastic">
+    <color rgba="0.1 0.1 0.1 1" />
+  </material>
+  <material name="zed_mat">
+    <color rgba="0.8 0.8 0.8 1.0" />
+  </material>
+  <material name="zedm_mat">
+    <color rgba="0 0 0 1.0" />
+  </material>
+  <material name="zed2_mat">
+    <color rgba="0.25 0.25 0.25 1.0" />
+  </material>
+  <material name="zed2i_mat">
+    <color rgba="0.25 0.25 0.25 1.0" />
+  </material>
+  <material name="zedx_mat">
+    <color rgba="0.25 0.25 0.25 1.0" />
+  </material>
+  <material name="zedxm_mat">
+    <color rgba="0.25 0.25 0.25 1.0" />
+  </material>
+  <material name="virtual_mat">
+    <color rgba="0.25 0.25 0.25 1.0" />
+  </material>
+  <material name="zedxonegs_mat">
+    <color rgba="0.25 0.25 0.25 1.0" />
+  </material>
+  <material name="zedxone4k_mat">
+    <color rgba="0.25 0.25 0.25 1.0" />
   </material>
 </robot>
