Commit message: added isaac files and ino

File: src/grr_description/grreg.urdf (robot description, URDF)
Before this commit: robot bloodstone, 55 links, 54 joints
Links:
- link front_left_mecanum_link: geometry collision cylinder length=0.042 radius=0.030015; visual mesh filename=package://grr_description/meshes/mecanum_wheel_1.stl scale=0.001 0.001 0.001
- link front_right_mecanum_link: geometry collision cylinder length=0.042 radius=0.030015; visual mesh filename=package://grr_description/meshes/mecanum_wheel_2.stl scale=0.001 0.001 0.001
- link rear_left_mecanum_link: geometry collision cylinder length=0.042 radius=0.030015; visual mesh filename=package://grr_description/meshes/mecanum_wheel_2.stl scale=0.001 0.001 0.001
- link rear_right_mecanum_link: geometry collision cylinder length=0.042 radius=0.030015; visual mesh filename=package://grr_description/meshes/mecanum_wheel_1.stl scale=0.001 0.001 0.001
Joints:
- joint front_left_mecanum_joint: axis 0.0 -1.0 0.0  -> 0.0 1.0 0.0 ; origin xyz=-0.10075 0.10075 0 rpy=0 1.5707963267948966 0 -> xyz=0.09 0.10075 0 rpy=0 -1.5707963267948966 0
- joint front_left_roller_0_joint: origin xyz=0.0 0 0.030015 rpy=0.0 0 0.7853981633974483 -> xyz=0.0 0 0.030015 rpy=-0.0 0 -0.7853981633974483
- joint front_left_roller_1_joint: origin xyz=0.02122381003731422 0 0.021223810037314224 rpy=0.5553603672697958 0 0.5553603672697958 -> xyz=0.02122381003731422 0 0.021223810037314224 rpy=-0.5553603672697958 0 -0.5553603672697958
- joint front_left_roller_2_joint: origin xyz=0.030015 0 1.8378886838203904e-18 rpy=0.7853981633974483 0 4.8091767343044744e-17 -> xyz=0.030015 0 1.8378886838203904e-18 rpy=-0.7853981633974483 0 -4.8091767343044744e-17
- joint front_left_roller_3_joint: origin xyz=0.021223810037314224 0 -0.02122381003731422 rpy=0.5553603672697958 0 -0.5553603672697958 -> xyz=0.021223810037314224 0 -0.02122381003731422 rpy=-0.5553603672697958 0 0.5553603672697958
- joint front_left_roller_4_joint: origin xyz=3.675777367640781e-18 0 -0.030015 rpy=9.618353468608949e-17 0 -0.7853981633974483 -> xyz=3.675777367640781e-18 0 -0.030015 rpy=-9.618353468608949e-17 0 0.7853981633974483
- joint front_left_roller_5_joint: origin xyz=-0.02122381003731422 0 -0.021223810037314227 rpy=-0.5553603672697958 0 -0.5553603672697959 -> xyz=-0.02122381003731422 0 -0.021223810037314227 rpy=0.5553603672697958 0 0.5553603672697959
- joint front_left_roller_6_joint: origin xyz=-0.030015 0 -5.513666051461171e-18 rpy=-0.7853981633974483 0 -1.4427530202913423e-16 -> xyz=-0.030015 0 -5.513666051461171e-18 rpy=0.7853981633974483 0 1.4427530202913423e-16
- joint front_left_roller_7_joint: origin xyz=-0.021223810037314227 0 0.02122381003731422 rpy=-0.5553603672697959 0 0.5553603672697957 -> xyz=-0.021223810037314227 0 0.02122381003731422 rpy=0.5553603672697959 0 -0.5553603672697957
- joint front_right_mecanum_joint: axis 0.0 -1.0 0.0  -> 0.0 1.0 0.0 ; origin xyz=0.10075 0.10075 0 rpy=0 1.5707963267948966 0 -> xyz=0.09 -0.10075 0 rpy=0 -1.5707963267948966 0
- joint front_right_roller_0_joint: origin xyz=0.0 0 0.030015 rpy=-0.0 0 -0.7853981633974483 -> xyz=0.0 0 0.030015 rpy=0.0 0 0.7853981633974483
- joint front_right_roller_1_joint: origin xyz=0.02122381003731422 0 0.021223810037314224 rpy=-0.5553603672697958 0 -0.5553603672697958 -> xyz=0.02122381003731422 0 0.021223810037314224 rpy=0.5553603672697958 0 0.5553603672697958
- joint front_right_roller_2_joint: origin xyz=0.030015 0 1.8378886838203904e-18 rpy=-0.7853981633974483 0 -4.8091767343044744e-17 -> xyz=0.030015 0 1.8378886838203904e-18 rpy=0.7853981633974483 0 4.8091767343044744e-17
- joint front_right_roller_3_joint: origin xyz=0.021223810037314224 0 -0.02122381003731422 rpy=-0.5553603672697958 0 0.5553603672697958 -> xyz=0.021223810037314224 0 -0.02122381003731422 rpy=0.5553603672697958 0 -0.5553603672697958
- joint front_right_roller_4_joint: origin xyz=3.675777367640781e-18 0 -0.030015 rpy=-9.618353468608949e-17 0 0.7853981633974483 -> xyz=3.675777367640781e-18 0 -0.030015 rpy=9.618353468608949e-17 0 -0.7853981633974483
- joint front_right_roller_5_joint: origin xyz=-0.02122381003731422 0 -0.021223810037314227 rpy=0.5553603672697958 0 0.5553603672697959 -> xyz=-0.02122381003731422 0 -0.021223810037314227 rpy=-0.5553603672697958 0 -0.5553603672697959
- joint front_right_roller_6_joint: origin xyz=-0.030015 0 -5.513666051461171e-18 rpy=0.7853981633974483 0 1.4427530202913423e-16 -> xyz=-0.030015 0 -5.513666051461171e-18 rpy=-0.7853981633974483 0 -1.4427530202913423e-16
- joint front_right_roller_7_joint: origin xyz=-0.021223810037314227 0 0.02122381003731422 rpy=0.5553603672697959 0 -0.5553603672697957 -> xyz=-0.021223810037314227 0 0.02122381003731422 rpy=-0.5553603672697959 0 0.5553603672697957
- joint left_bin_grabber_finger_joint: axis 0 0 1 -> 0 -1 0; limit (none) -> lower=-3.14 upper=0.39 effort=10 velocity=0.5; type continuous -> revolute
- joint left_bin_grabber_pivot_joint: axis 0 0 1 -> 0 1 0; limit (none) -> lower=-0.39 upper=0.044 effort=10 velocity=0.5; type continuous -> revolute
- joint rear_left_mecanum_joint: origin xyz=-0.10075 -0.10075 0 rpy=0 -1.5707963267948966 0 -> xyz=-0.09 0.10075 0 rpy=0 -1.5707963267948966 0
- joint rear_left_roller_0_joint: origin xyz=0.0 0 0.030015 rpy=-0.0 0 -0.7853981633974483 -> xyz=0.0 0 0.030015 rpy=0.0 0 0.7853981633974483
- joint rear_left_roller_1_joint: origin xyz=0.02122381003731422 0 0.021223810037314224 rpy=-0.5553603672697958 0 -0.5553603672697958 -> xyz=0.02122381003731422 0 0.021223810037314224 rpy=0.5553603672697958 0 0.5553603672697958
- joint rear_left_roller_2_joint: origin xyz=0.030015 0 1.8378886838203904e-18 rpy=-0.7853981633974483 0 -4.8091767343044744e-17 -> xyz=0.030015 0 1.8378886838203904e-18 rpy=0.7853981633974483 0 4.8091767343044744e-17
- joint rear_left_roller_3_joint: origin xyz=0.021223810037314224 0 -0.02122381003731422 rpy=-0.5553603672697958 0 0.5553603672697958 -> xyz=0.021223810037314224 0 -0.02122381003731422 rpy=0.5553603672697958 0 -0.5553603672697958
- joint rear_left_roller_4_joint: origin xyz=3.675777367640781e-18 0 -0.030015 rpy=-9.618353468608949e-17 0 0.7853981633974483 -> xyz=3.675777367640781e-18 0 -0.030015 rpy=9.618353468608949e-17 0 -0.7853981633974483
- joint rear_left_roller_5_joint: origin xyz=-0.02122381003731422 0 -0.021223810037314227 rpy=0.5553603672697958 0 0.5553603672697959 -> xyz=-0.02122381003731422 0 -0.021223810037314227 rpy=-0.5553603672697958 0 -0.5553603672697959
- joint rear_left_roller_6_joint: origin xyz=-0.030015 0 -5.513666051461171e-18 rpy=0.7853981633974483 0 1.4427530202913423e-16 -> xyz=-0.030015 0 -5.513666051461171e-18 rpy=-0.7853981633974483 0 -1.4427530202913423e-16
- joint rear_left_roller_7_joint: origin xyz=-0.021223810037314227 0 0.02122381003731422 rpy=0.5553603672697959 0 -0.5553603672697957 -> xyz=-0.021223810037314227 0 0.02122381003731422 rpy=-0.5553603672697959 0 0.5553603672697957
- joint rear_right_mecanum_joint: origin xyz=0.10075 -0.10075 0 rpy=0 -1.5707963267948966 0 -> xyz=-0.09 -0.10075 0 rpy=0 -1.5707963267948966 0
- joint rear_right_roller_0_joint: origin xyz=0.0 0 0.030015 rpy=0.0 0 0.7853981633974483 -> xyz=0.0 0 0.030015 rpy=-0.0 0 -0.7853981633974483
- joint rear_right_roller_1_joint: origin xyz=0.02122381003731422 0 0.021223810037314224 rpy=0.5553603672697958 0 0.5553603672697958 -> xyz=0.02122381003731422 0 0.021223810037314224 rpy=-0.5553603672697958 0 -0.5553603672697958
- joint rear_right_roller_2_joint: origin xyz=0.030015 0 1.8378886838203904e-18 rpy=0.7853981633974483 0 4.8091767343044744e-17 -> xyz=0.030015 0 1.8378886838203904e-18 rpy=-0.7853981633974483 0 -4.8091767343044744e-17
- joint rear_right_roller_3_joint: origin xyz=0.021223810037314224 0 -0.02122381003731422 rpy=0.5553603672697958 0 -0.5553603672697958 -> xyz=0.021223810037314224 0 -0.02122381003731422 rpy=-0.5553603672697958 0 0.5553603672697958
- joint rear_right_roller_4_joint: origin xyz=3.675777367640781e-18 0 -0.030015 rpy=9.618353468608949e-17 0 -0.7853981633974483 -> xyz=3.675777367640781e-18 0 -0.030015 rpy=-9.618353468608949e-17 0 0.7853981633974483
- joint rear_right_roller_5_joint: origin xyz=-0.02122381003731422 0 -0.021223810037314227 rpy=-0.5553603672697958 0 -0.5553603672697959 -> xyz=-0.02122381003731422 0 -0.021223810037314227 rpy=0.5553603672697958 0 0.5553603672697959
- joint rear_right_roller_6_joint: origin xyz=-0.030015 0 -5.513666051461171e-18 rpy=-0.7853981633974483 0 -1.4427530202913423e-16 -> xyz=-0.030015 0 -5.513666051461171e-18 rpy=0.7853981633974483 0 1.4427530202913423e-16
- joint rear_right_roller_7_joint: origin xyz=-0.021223810037314227 0 0.02122381003731422 rpy=-0.5553603672697959 0 0.5553603672697957 -> xyz=-0.021223810037314227 0 0.02122381003731422 rpy=0.5553603672697959 0 -0.5553603672697957
- joint right_bin_grabber_finger_joint: axis 0 0 1 -> 0 1 0; limit (none) -> lower=-3.14 upper=0.39 effort=10 velocity=0.5; type continuous -> revolute
- joint right_bin_grabber_pivot_joint: axis 0 0 1 -> 0 1 0; limit (none) -> lower=-0.39 upper=0.044 effort=10 velocity=0.5; type continuous -> revolute

File: src/grr_description/urdf/parts/bin_grabber.xacro (robot description, xacro)
@@ -37,9 +37,10 @@
         </collision>
     </link>
-    <joint name="${prefix}_bin_grabber_pivot_joint" type="continuous">
+    <joint name="${prefix}_bin_grabber_pivot_joint" type="revolute">
         <parent link="${prefix}_bin_grabber_base_link"/>
         <child link="${prefix}_bin_grabber_pivot_link"/>
         <origin xyz="0.0 0.005 0" rpy="0 0 0"/>
-        <axis xyz="0 0 1"/>
+        <axis xyz="0 1 0"/>
+        <limit lower="-0.35" upper="0.044" effort="10" velocity="0.5"/>
     </joint>
     <link name="${prefix}_bin_grabber_finger_link">
@@ -58,9 +59,11 @@
         </collision>
     </link>
-    <joint name="${prefix}_bin_grabber_finger_joint" type="continuous">
+    <joint name="${prefix}_bin_grabber_finger_joint" type="revolute">
         <parent link="${prefix}_bin_grabber_pivot_link"/>
         <child link="${prefix}_bin_grabber_finger_link"/>
         <origin xyz="${0.01*reverse} 0.002 0.06" rpy="0 0 0"/>
-        <axis xyz="0 0 1"/>
+        <axis xyz="0 ${reverse} 0"/>
+        <!-- add joint limits -->
+        <limit lower="-3.14" upper="0.39" effort="10" velocity="0.5"/>
     </joint>
 </xacro:macro>

File: src/grr_description/urdf/robots/grreg.urdf.xacro (robot description, xacro)
@@ -21,5 +21,5 @@
   <xacro:property name="wheel_weight" value="0.136" />
   <xacro:property name="wheel_offset" value="0" />
-  <xacro:property name="wheel_joint_pos_x" value="0.10075" />
+  <xacro:property name="wheel_joint_pos_x" value="0.09" />
   <xacro:property name="wheel_joint_pos_y" value="0.10075" />
   <xacro:property name="wheel_joint_pos_z" value="0.07793" />
@@ -36,9 +36,9 @@
   </xacro:chassis>
   <xacro:mecanum_with_rollers
-    name="front_right"
+    name="front_left"
     type="1"
     radius="${wheel_radius}"
     width="${wheel_thickness}"
-    flip="${pi/2}"
+    flip="-${pi/2}"
     pos_x="${wheel_joint_pos_x + wheel_offset}"
     pos_y="${wheel_joint_pos_y}"
@@ -47,5 +47,5 @@
   />
   <xacro:mecanum_with_rollers
-    name="rear_left"
+    name="rear_right"
     type="1"
     radius="${wheel_radius}"
@@ -58,9 +58,9 @@
   />
   <xacro:mecanum_with_rollers
-    name="front_left"
+    name="rear_left"
     type="2"
     radius="${wheel_radius}"
     width="${wheel_thickness}"
-    flip="${pi/2}"
+    flip="-${pi/2}"
     pos_x="-${wheel_joint_pos_x + wheel_offset}"
     pos_y="${wheel_joint_pos_y}"
@@ -69,5 +69,5 @@
   />
   <xacro:mecanum_with_rollers
-    name="rear_right"
+    name="front_right"
     type="2"
     radius="${wheel_radius}"

Commit message: fixed urdf problems

File: src/grr_description/grreg.urdf (robot description, URDF)
Before this commit: robot bloodstone, 55 links, 54 joints
Joints:
- joint left_bin_grabber_pivot_joint: limit lower=-0.39 upper=0.044 effort=10 velocity=0.5 -> lower=-0.35 upper=0.044 effort=10 velocity=0.5
- joint right_bin_grabber_pivot_joint: limit lower=-0.39 upper=0.044 effort=10 velocity=0.5 -> lower=-0.35 upper=0.044 effort=10 velocity=0.5

File: src/grr_description/urdf/control/drive.xacro (robot description, xacro)
@@ -3,7 +3,81 @@
   <ros2_control name="bloodstone" type="system">
     <hardware>
-      <plugin>grr_hardware/IsaacDriveHardware</plugin>
+      <plugin>grr_hardware/CanInterface</plugin>
       <param name="example_param_hw_start_duration_sec">3.0</param>
       <param name="example_param_hw_stop_duration_sec">3.0</param>
+      <param name="teensy1_serial_number">3030313330356332</param>
+      <param name="teensy1_joint_names">
+        <item>front_right_mecanum_joint</item>
+        <item>front_left_mecanum_joint</item>
+      </param>
+      <param name="front_right_mecanum_joint">
+        <item name="DIR">1</item>
+        <item name="PWM">2</item>
+        <item name="SLP">7</item>
+        <item name="FLT">8</item>
+        <item name="ENC_OUTA">11</item>
+        <item name="ENC_OUTB">12</item>
+        <item name="CS">23</item>
+      </param>
+      <param name="front_left_mecanum_joint">
+        <item name="DIR">29</item>
+        <item name="PWM">28</item>
+        <item name="SLP">34</item>
+        <item name="FLT">35</item>
+        <item name="ENC_OUTA">24</item>
+        <item name="ENC_OUTB">25</item>
+        <item name="CS">40</item>
+      </param>
+      <param name="teensy2_joint_names">
+        <item>rear_right_mecanum_joint</item>
+        <item>rear_left_mecanum_joint</item>
+        <item>intake_roller_1_joint</item>
+        <item>intake_roller_2_joint</item>
+        <item>sorter_turntable_joint</item>
+        <item>left_bin_grabber_pivot_joint</item>
+        <item>left_bin_grabber_finger_joint</item>
+        <item>right_bin_grabber_pivot_joint</item>
+        <item>right_bin_grabber_finger_joint</item>
+      </param>
+      <param name="rear_right_mecanum_joint">
+        <item name="DIR">1</item>
+        <item name="PWM">2</item>
+        <item name="SLP">7</item>
+        <item name="FLT">8</item>
+        <item name="ENC_OUTA">11</item>
+        <item name="ENC_OUTB">12</item>
+        <item name="CS">23</item>
+      </param>
+      <param name="rear_left_mecanum_joint">
+        <item name="DIR">29</item>
+        <item name="PWM">28</item>
+        <item name="SLP">34</item>
+        <item name="FLT">35</item>
+        <item name="ENC_OUTA">24</item>
+        <item name="ENC_OUTB">25</item>
+        <item name="CS">40</item>
+      </param>
+      <param name="intake_roller_1_joint">
+        <item name="PWM">36</item>
+      </param>
+      <param name="intake_roller_2_joint">
+        <item name="PWM">37</item>
+      </param>
+      <param name="sorter_turntable_joint">
+        <item name="PWM">3</item>
+      </param>
+      <param name="left_bin_grabber_pivot_joint">
+        <item name="PWM">4</item>
+      </param>
+      <param name="left_bin_grabber_finger_joint">
+        <item name="PWM">5</item>
+      </param>
+      <param name="right_bin_grabber_pivot_joint">
+        <item name="PWM">6</item>
+      </param>
+      <param name="right_bin_grabber_finger_joint">
+        <item name="PWM">9</item>
+      </param>
+      <param name="teensy2_serial_number">3030313330356332</param>
     </hardware>
     <joint name="front_right_mecanum_joint">
@@ -39,11 +113,36 @@
       <state_interface name="velocity"/>
     </joint>
-    <joint name="small_package_grabber_roller_1_joint">
-      <command_interface name="effort"/>
+    <joint name="intake_roller_1_joint">
+      <command_interface name="effor"/>
       <state_interface name="position"/>
       <state_interface name="velocity"/>
     </joint>
-    <joint name="small_package_sweeper_roller_joint">
-      <command_interface name="effort"/>
+    <joint name="intake_roller_2_joint">
+      <command_interface name="effor"/>
+      <state_interface name="position"/>
+      <state_interface name="velocity"/>
+    </joint>
+    <joint name="sorter_turntable_joint">
+      <command_interface name="effor"/>
+      <state_interface name="position"/>
+      <state_interface name="velocity"/>
+    </joint>
+    <joint name="left_bin_grabber_pivot_joint">
+      <command_interface name="position"/>
+      <state_interface name="position"/>
+      <state_interface name="velocity"/>
+    </joint>
+    <joint name="left_bin_grabber_finger_joint">
+      <command_interface name="position"/>
+      <state_interface name="position"/>
+      <state_interface name="velocity"/>
+    </joint>
+    <joint name="right_bin_grabber_pivot_joint">
+      <command_interface name="position"/>
+      <state_interface name="position"/>
+      <state_interface name="velocity"/>
+    </joint>
+    <joint name="right_bin_grabber_finger_joint">
+      <command_interface name="position"/>
       <state_interface name="position"/>
       <state_interface name="velocity"/>
